File: custom_altimeter.kicad_sch (KiCad schematic)
At the start: 4 parts, among them U1 Pico

Commit message: Changes for 2024
Parts:
- removed U1: Pico, Library:RPi_Pico_SMD_TH, symbol Local:Pico
- added U1: FEATHERWING_NODIM, Library:FEATHERWING_NODIM, symbol NRF52840:FEATHERWING_NODIM
