File: custom_altimeter.kicad_pcb (KiCad board)
At the start: 2 copper layers, 4 parts, among them U1 Pico

Commit message: Changes for 2024
Parts:
- U1: value Pico -> FEATHERWING_NODIM; footprint Library:RPi_Pico_SMD_TH -> Library:FEATHERWING_NODIM; moved to B.Cu
- moved U1 6.26 mm to (96.5, 129.3), turned to 180 degrees

Commit message: Additional fixes
Parts:
- U1: moved to F.Cu
- moved U1 47.9 mm to (48.7, 127.3), turned to 0 degrees
